File: hardware/proto40/power.kicad_sch (KiCad schematic)
At the start: 26 parts, among them J101 USB_C_Receptacle_USB2.0_16P, Q101 BCP53, U101 USBLC6-2SC6, U102 LM66100DCK, U103 TL431DBZ, U104 AP2112K-3.3

Commit message: Redraw Proto40 schematic with wired functional blocks
Review feedback: text overlapped components and parts were isolated
islands joined only by labels, so connectivity was hard to follow.

- Generator: polyline wires, automatic junctions, text placement from
  the real symbol body graphics, KiCad field-angle handling for rotated
  symbols, power symbols oriented normally on horizontal pins
- Sheets redrawn left-to-right with wired blocks: channel cells, BIAS
  rail, decoupling on IC power pins, pull-ups on their lines, control
  ladder across the six groups, visible 165 chain, wired root hierarchy
  (MCU -> Control -> both sides) and cross-side LOOP
- layoutcheck.py: rejects text/text, text/body, text/wire overlaps and
  wires through bodies; CI runs the generator with --strict
- check_proto40.py: finds parts by sheet path and follows pins, so it no
  longer depends on net names or reference numbering

ERC 0 violations, design-intent audit PASS, layout issues 0.

Co-Authored-By: Claude Opus 5.5 <noreply@anthropic.com>
Claude-Session: https://claude.ai/code/session_01UG7pR5ZtgvoVGRWFojzQKf
Parts:
- C101: Note shield to GND, ≥ 100 V -> ≥ 100 V
- C104: value 100n -> 10u; footprint Capacitor_SMD:C_0603_1608Metric -> Capacitor_SMD:C_0805_2012Metric
- C105: value 10u -> 100n; footprint Capacitor_SMD:C_0805_2012Metric -> Capacitor_SMD:C_0603_1608Metric
- R107: Note sets clamp at ≈ 5.45 V -> sets clamp ≈ 5.45 V
Connections:
- net +3V3: now also C107.1; no longer C106.1
- net USB_DM: now also U101.6 (I/O1); no longer U101.4 (I/O2)
- net USB_DP: now also U101.4 (I/O2); no longer U101.6 (I/O1)
- net VBUS_F: now also C102.1; no longer C105.1
- net VDD5: now also C105.1, C106.1; no longer C102.1, C107.1
- net CLAMP_C: no longer names the net of Q101.2 (C), Q101.4 (C), R104.1
- net CLAMP_K: no longer names the net of R106.2, U103.1 (K)
- net CLAMP_REF: no longer names the net of R107.2, R108.1, U103.2 (REF)
- net USB_D+: no longer names the net of J101.A6 (D+), J101.B6 (D+)
- net USB_D+: now also U101.3 (I/O2); no longer U101.1 (I/O1)
- net USB_D-: no longer names the net of J101.A7 (D-), J101.B7 (D-)
- net USB_D-: now also U101.1 (I/O1); no longer U101.3 (I/O2)
- net USB_SHIELD: no longer names the net of C101.1, J101.SH (SHIELD), R103.1
- net VDD5_RAW: no longer names the net of FB101.1, U102.6 (VOUT)
Other:
- note added: "VBUS -> PTC -> LM66100 ideal diode (never back-feeds the host) -> ferrite -> VDD5. TL431 + BCP53 shunt clamp holds VDD5 <= 5.45 V when fixture faults inject current (review F9)."
- note removed: "VBUS → polyfuse → LM66100 (reverse blocking, never back-feeds the host) → ferrite → VDD5. TL431 + BCP53 shunt clamp holds VDD5 ≤ 5.45 V when fixture faults inject current (review F9)."
- moved on the sheet: C101, C102, C103, C104, C105, C106, C107, F101, FB101, J101, Q101, R101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
