File: hardware/proto40/control.kicad_sch (KiCad schematic)
At the start: 19 parts, among them U301 74AHCT125, U302 74AHCT125, U303 74LVC1G125, U304 74AHCT1G125

Commit message: Resolve Proto40 house-style review findings
- Fixture ID lines: TVS at the connector plus series R on SDA/SCL/WP/A0/PRESENT_N;
  ID_VCC limited by 100 ohm 1206 (D14). PRESENT_N pull-up moved to MCU side.
- Shunt clamp ballast R104 is 6.8 ohm 2512, BCP53 copper note (D15).
- MPN/Manufacturer on every part (generic Yageo/Samsung passives), LCSC TBD.
- Test points on the '595 outputs and chain in/out; pull-downs on SCK/RCLK.
- Root sheet: CTRL/SENSE chains and ID lines drawn as wires; ASCII-only text.
- layoutcheck: non-ASCII, title length, text/text gap, text/wire clearance,
  NC flag on wired pin; wider char estimate. CI ERC runs --severity-all.
- Netclass patterns tightened for STIM/MUX and SPI nets.

Co-Authored-By: Claude Opus 5.5 (1M context) <noreply@anthropic.com>
Claude-Session: https://claude.ai/code/session_013SDanWEFU4wFXEYfZ6C9GH
Parts:
- added R309, R310: 100k, Resistor_SMD:R_0603_1608Metric, symbol Device:R
- C301, C302, C303, C304: LCSC (none) -> TBD; MPN (none) -> CL10B104KB8NNNC; Manufacturer (none) -> Samsung Electro-Mechanics
- C305, C306: LCSC (none) -> TBD; MPN (none) -> CL10B102KB8NNNC; Manufacturer (none) -> Samsung Electro-Mechanics
- R301, R302: value 10k -> 100k; LCSC (none) -> TBD; MPN (none) -> RC0603FR-07100KL; Manufacturer (none) -> Yageo; Note inactive during MCU reset -> no clock edges during MCU reset
- R303: LCSC (none) -> TBD; MPN (none) -> RC0603FR-0710KL; Manufacturer (none) -> Yageo; Note stimulus off during MCU reset -> inactive during MCU reset
- R304: value 150 -> 10k; LCSC (none) -> TBD; MPN (none) -> RC0603FR-0710KL; Manufacturer (none) -> Yageo; Note Rlim -> inactive during MCU reset
- R305: value 100k -> 10k; LCSC (none) -> TBD; MPN (none) -> RC0603FR-0710KL; Manufacturer (none) -> Yageo; Note (none) -> stimulus off during MCU reset
- R306: value 100k -> 150; LCSC (none) -> TBD; MPN (none) -> RC0603FR-07150RL; Manufacturer (none) -> Yageo; Note (none) -> Rlim
- R307, R308: LCSC (none) -> TBD; MPN (none) -> RC0603FR-07100KL; Manufacturer (none) -> Yageo
- TP301: LCSC (none) -> none; MPN (none) -> none (PCB pad only)
- U301, U302, U303, U304: LCSC (none) -> TBD
Connections:
- net +3V3: now also R304.1, R305.1; no longer R301.1, R302.1
- net ADC_STIM: now also R307.2, R308.1; no longer R305.2, R306.1
- net ADC_VDD5: now also R309.2, R310.1; no longer R307.2, R308.1
- net BIAS_EN_N: now also R304.2; no longer R302.2
- net GND: now also R301.2, R302.2, R310.2; no longer R306.2
- net OE_N: now also R303.2; no longer R301.2
- net RCLK: now also R302.1
- net SCK: now also R301.1
- net STIM: now also R306.2, R307.1; no longer R304.2, R305.1
- net STIM_EN_N: now also R305.2; no longer R303.2
- net VDD5: now also R309.1; no longer R307.1
- net at U304.4: now also R306.1; no longer R304.1
Other:
- note added: "MCU (3.3 V) -> 5 V logic: 74AHCT125 (TTL input levels). 5 V sense chain -> MCU: 74LVC1G125 at 3.3 V. Pull-ups keep OE5_N, BIAS_EN and STIM_EN inactive while the MCU is in reset (review F6); pull-downs keep SCK and RCLK from clocking the chain while the MCU pins float."
- note removed: "MCU (3.3 V) -> 5 V logic: 74AHCT125 (TTL input levels). 5 V sense chain -> MCU: 74LVC1G125 at 3.3 V. Pull-ups keep OE5_N, BIAS_EN and STIM_EN inactive while the MCU is in reset (review F6)."
- title: Proto40 – level shifting, stimulus driver, ADC taps -> Proto40 - level shifting, stimulus driver, ADC taps
- moved on the sheet: R301, R302, R303, R304, R305, R306, R307, R308
