File: hardware/proto40/side.kicad_sch (KiCad schematic)
At the start: 18 parts, among them J1001 DIN41612_02x32_AC, U1001 74HC595, U1002 TMUX1308, U1003 74AHCT1G125

Commit message: Resolve Proto40 house-style review findings
- Fixture ID lines: TVS at the connector plus series R on SDA/SCL/WP/A0/PRESENT_N;
  ID_VCC limited by 100 ohm 1206 (D14). PRESENT_N pull-up moved to MCU side.
- Shunt clamp ballast R104 is 6.8 ohm 2512, BCP53 copper note (D15).
- MPN/Manufacturer on every part (generic Yageo/Samsung passives), LCSC TBD.
- Test points on the '595 outputs and chain in/out; pull-downs on SCK/RCLK.
- Root sheet: CTRL/SENSE chains and ID lines drawn as wires; ASCII-only text.
- layoutcheck: non-ASCII, title length, text/text gap, text/wire clearance,
  NC flag on wired pin; wider char estimate. CI ERC runs --severity-all.
- Netclass patterns tightened for STIM/MUX and SPI nets.

Co-Authored-By: Claude Opus 5.5 (1M context) <noreply@anthropic.com>
Claude-Session: https://claude.ai/code/session_013SDanWEFU4wFXEYfZ6C9GH
Parts:
- added D1001, D1002, D1003, D1004, D1005, D1006: ESD 5V, Diode_SMD:D_SOD-323, symbol Device:D_TVS
- added R1009, R1010: 220, Resistor_SMD:R_0603_1608Metric, symbol Device:R
- added R1011, R1012: 1k, Resistor_SMD:R_0603_1608Metric, symbol Device:R
- added R1013: 100, Resistor_SMD:R_1206_3216Metric, symbol Device:R
- added TP1002: SENSE_OUT, TestPoint:TestPoint_Pad_D1.0mm, symbol Connector:TestPoint
- added TP1003: CTRL_IN, TestPoint:TestPoint_Pad_D1.0mm, symbol Connector:TestPoint
- added TP1004: CTRL_OUT, TestPoint:TestPoint_Pad_D1.0mm, symbol Connector:TestPoint
- added TP1005: BIAS_RAIL, TestPoint:TestPoint_Pad_D1.0mm, symbol Connector:TestPoint
- added TP1006: ADDR1_0, TestPoint:TestPoint_Pad_D1.0mm, symbol Connector:TestPoint
- added TP1007: ADDR1_1, TestPoint:TestPoint_Pad_D1.0mm, symbol Connector:TestPoint
- added TP1008: ADDR1_2, TestPoint:TestPoint_Pad_D1.0mm, symbol Connector:TestPoint
- added TP1009: ADDR2_0, TestPoint:TestPoint_Pad_D1.0mm, symbol Connector:TestPoint
- added TP1010: ADDR2_1, TestPoint:TestPoint_Pad_D1.0mm, symbol Connector:TestPoint
- added TP1011: ADDR2_2, TestPoint:TestPoint_Pad_D1.0mm, symbol Connector:TestPoint
- added TP1012: EN2_N, TestPoint:TestPoint_Pad_D1.0mm, symbol Connector:TestPoint
- added TP1013: BIAS, TestPoint:TestPoint_Pad_D1.0mm, symbol Connector:TestPoint
- C1001, C1003, C1004, C1005: LCSC (none) -> TBD; MPN (none) -> CL10B104KB8NNNC; Manufacturer (none) -> Samsung Electro-Mechanics
- C1002: LCSC (none) -> TBD; MPN (none) -> CL21A106KAYNNNE; Manufacturer (none) -> Samsung Electro-Mechanics
- J1001: LCSC (none) -> TBD; MPN DIN 41612 type C 2x32 female vertical, performance level 1/2 -> TBD: DIN 41612 type C 2x32 female vertical, performance lev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
- R1001: value 10k -> 100k; LCSC (none) -> TBD; MPN (none) -> RC0603FR-07100KL; Manufacturer (none) -> Yageo; Note (none) -> load-signature reference node
- R1002: LCSC (none) -> TBD; MPN (none) -> RC0603FR-07100KL; Manufacturer (none) -> Yageo; Note load-signature reference node -> mux off while 595 outputs are Hi-Z
- R1003: LCSC (none) -> TBD; MPN (none) -> RC0603FR-07100KL; Manufacturer (none) -> Yageo; Note mux off while 595 outputs are Hi-Z -> (none)
- R1004: LCSC (none) -> TBD; MPN (none) -> RC0603FR-07100KL; Manufacturer (none) -> Yageo
- R1005: LCSC (none) -> TBD; MPN (none) -> RC0603FR-07100KL; Manufacturer (none) -> Yageo; Note (none) -> bias low while 595 outputs are Hi-Z
- R1006: LCSC (none) -> TBD; MPN (none) -> RC0603FR-07100KL; Manufacturer (none) -> Yageo; Note bias low while 595 outputs are Hi-Z -> bias Hi-Z until the MCU enables it
- R1007: value 100k -> 1k; LCSC (none) -> TBD; MPN (none) -> RC0603FR-071KL; Manufacturer (none) -> Yageo; Note bias Hi-Z until the MCU enables it -> series R, fixture ID line
- R1008: value 47 -> 10k; LCSC (none) -> TBD; MPN (none) -> RC0603FR-0710KL; Manufacturer (none) -> Yageo; Note ID_VCC current limit -> adapter ties PRESENT_N to GND
- TP1001: value BIAS_RAIL -> SENSE_IN; LCSC (none) -> none; MPN (none) -> none (PCB pad only)
- U1001, U1003: LCSC (none) -> TBD
- U1002: LCSC (none) -> TBD; MPN (none) -> TMUX1308PWR; Manufacturer (none) -> Texas Instruments
Connections:
- net +3V3: now also R1013.1; no longer R1001.1
- net ADDR1_0: now also TP1006.1
- net ADDR1_1: now also TP1007.1
- net ADDR1_2: now also TP1008.1
- net ADDR2_0: now also TP1009.1
- net ADDR2_1: now also TP1010.1
- net ADDR2_2: now also TP1011.1
- net BIAS: now also R1005.1, TP1013.1; no longer R1006.1
- net BIAS_EN_N: now also R1006.2; no longer R1007.2
- net BIAS_RAIL: now also TP1005.1; no longer TP1001.1
- net CTRL_IN: now also TP1003.1
- net CTRL_OUT: now also TP1004.1
- net EN2_N: now also R1002.2, TP1012.1; no longer R1003.2
- net G6/EXT3: now also R1001.1; no longer R1002.1
- net GND: now also R1001.2, R1004.2, D1001.1 (A1), D1002.1 (A1), D1003.1 (A1), D1004.1 (A1), D1005.1 (A1), D1006.1 (A1); no longer R1002.2, R1006.2
- net ID_A0: now also R1012.2; no longer J1001.c30 (Pin_c30)
- net ID_SCL: now also R1010.2; no longer J1001.a30 (Pin_a30)
- net ID_SDA: now also R1009.2; no longer J1001.a29 (Pin_a29)
- net ID_WP: now also R1011.2; no longer J1001.c29 (Pin_c29)
- net PRESENT_N: now also R1007.2, R1008.2; no longer J1001.c28 (Pin_c28), R1001.2
- net SENSE_IN: now also TP1001.1
- net SENSE_OUT: now also TP1002.1
- net VDD5: now also R1002.1, R1006.1; no longer R1004.1, R1007.1
- net ID_VCC renamed ID_VCC_EXT
- net ID_VCC_EXT: now also D1006.2 (A2), R1013.2; no longer R1008.2
- removed net STIM_CAL: R1004.2, R1005.1, U1002.2 (S6)
- new net: R1003.2, R1004.1, U1002.2 (S6)
- new net ID_A0_EXT: D1005.2 (A2), J1001.c30 (Pin_c30), R1012.1
- new net ID_SCL_EXT: D1003.2 (A2), J1001.a30 (Pin_a30), R1010.1
- new net ID_SDA_EXT: D1002.2 (A2), J1001.a29 (Pin_a29), R1009.1
- new net ID_WP_EXT: D1004.2 (A2), J1001.c29 (Pin_c29), R1011.1
- new net PRESENT_N_EXT: D1001.2 (A2), J1001.c28 (Pin_c28), R1007.1
Other:
- note added: "Fixture ID lines: ESD diode at the connector side, then series R. Not rated for the 24 V node fault (D14)."
- note added: "Fixture connector pinout: docs/fixture-interface.md. EXT41-EXT50 not populated. G6 = internal nodes: SHELL, LOOP (wired to the other side), known-open, RREF (100 kOhm to GND)."
- note removed: "Fixture connector pinout: docs/fixture-interface.md. EXT41–EXT50 not populated on Proto40. G6 = internal nodes: SHELL, LOOP (wired to the other side), known-open, RREF (100 kOhm to GND)."
- title: Proto40 – bank side (fixture connector, 6 groups, 2nd-stage mux) -> Proto40 - bank side: connector, 6 groups, 2nd-stage mux
- moved on the sheet: C1005, R1001, R1002, R1003, R1004, R1005, R1006, R1007, R1008, TP1001
